File: sch/Z80proto-SAKI80/FDC_DMA.kicad_sch (KiCad schematic)
At the start: 40 parts, among them J301 FDD, Q301 A950, U301 HC138, U302 HC139, U304 AC74, U305 LH0083A, U306 TMS2793, U307 HC574, U308 LMC555, U309 HCU04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

Commit message: add SAKI80 support
add SAKI80(AKA Super AKI-80) support,
Modify Comand & intel HEX upload command to MiniLoader.
Connections:
- net IO0x*: no longer names the net of U301.15 (O0)
- net IO1x*: no longer names the net of U301.14 (O1)
- net IO2x*: no longer names the net of U301.13 (O2)
- net IO3x*: no longer names the net of U301.12 (O3)
- net IO5x*: no longer names the net of U301.10 (O5)
- net IO6x*: no longer names the net of U301.9 (O6)
- net IO7x*: no longer names the net of U301.7 (O7)
Changed lines of the file:
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@@
-    (stroke (width 0) (type default) (color 0 0 0 0))
-  )
-  (wire (pts (xy 148.59 57.15) (xy 160.02 57.15))
     (stroke (width 0) (type default) (color 0 0 0 0))
   )
@@
     (stroke (width 0) (type default) (color 0 0 0 0))
   )
-  (wire (pts (xy 148.59 62.23) (xy 160.02 62.23))
-    (stroke (width 0) (type default) (color 0 0 0 0))
-  )
   (wire (pts (xy 247.65 297.18) (xy 247.65 309.88))
     (stroke (width 0) (type default) (color 0 0 0 0))
@@
     (stroke (width 0) (type default) (color 0 0 0 0))
   )
-  (wire (pts (xy 148.59 49.53) (xy 160.02 49.53))
-    (stroke (width 0) (type default) (color 0 0 0 0))
-  )
   (wire (pts (xy 96.52 146.05) (xy 114.3 146.05))
     (stroke (width 0) (type default) (color 0 0 0 0))
@@
     (stroke (width 0) (type default) (color 0 0 0 0))
   )
-  (wire (pts (xy 148.59 44.45) (xy 160.02 44.45))
-    (stroke (width 0) (type default) (color 0 0 0 0))
-  )
   (wire (pts (xy 58.42 52.07) (xy 73.66 52.07))
     (stroke (width 0) (type default) (color 0 0 0 0))
@@
     (stroke (width 0) (type default) (color 0 0 0 0))
   )
-  (wire (pts (xy 148.59 46.99) (xy 160.02 46.99))
-    (stroke (width 0) (type default) (color 0 0 0 0))
-  )
   (wire (pts (xy 24.13 289.56) (xy 52.07 289.56))
     (stroke (width 0) (type default) (color 0 0 0 0))
   )
-  (wire (pts (xy 148.59 52.07) (xy 160.02 52.07))
-    (stroke (width 0) (type default) (color 0 0 0 0))
-  )
   (wire (pts (xy 24.13 275.59) (xy 52.07 275.59))
     (stroke (width 0) (type default) (color 0 0 0 0))
@@
     (stroke (width 0) (type default) (color 0 0 0 0))
   )
-  (wire (pts (xy 148.59 59.69) (xy 160.02 59.69))
-    (stroke (width 0) (type default) (color 0 0 0 0))
-  )
   (wire (pts (xy 240.03 359.41) (xy 241.3 359.41))
     (stroke (width 0) (type default) (color 0 0 0 0))
@@
     (effects (font (size 1.27 1.27)) (justify right bottom))
   )
-  (label "IO2x*" (at 151.13 49.53 0)
-    (effects (font (size 1.27 1.27)) (justify left bottom))
-  )
   (label "BUSφ" (at 26.67 153.67 0)
     (effects (font (size 1.27 1.27)) (justify left bottom))
@@
     (effects (font (size 1.27 1.27)) (justify right bottom))
   )
-  (label "IO1x*" (at 151.13 46.99 0)
-    (effects (font (size 1.27 1.27)) (justify left bottom))
-  )
   (label "D3" (at 186.69 95.25 0)
     (effects (font (size 1.27 1.27)) (justify left bottom))
@@
     (effects (font (size 1.27 1.27)) (justify left bottom))
   )
-  (label "IO3x*" (at 156.21 52.07 180)
-    (effects (font (size 1.27 1.27)) (justify right bottom))
-  )
   (label "D1" (at 40.64 62.23 0)
     (effects (font (size 1.27 1.27)) (justify left bottom))
@@
     (effects (font (size 1.27 1.27)) (justify left bottom))
   )
-  (label "IO7x*" (at 151.13 62.23 0)
-    (effects (font (size 1.27 1.27)) (justify left bottom))
-  )
   (label "M1*" (at 36.83 80.01 0)
     (effects (font (size 1.27 1.27)) (justify left bottom))
@@
     (effects (font (size 1.27 1.27)) (justify left bottom))
   )
-  (label "IO5x*" (at 151.13 57.15 0)
-    (effects (font (size 1.27 1.27)) (justify left bottom))
-  )
   (label "M_ON" (at 257.81 87.63 0)
     (effects (font (size 1.27 1.27)) (justify left bottom))
@@
     (effects (font (size 1.27 1.27)) (justify left bottom))
   )
-  (label "IO6x*" (at 151.13 59.69 0)
-    (effects (font (size 1.27 1.27)) (justify left bottom))
-  )
   (label "A12" (at 80.01 148.59 180)
     (effects (font (size 1.27 1.27)) (justify right bottom))
@@
     (effects (font (size 1.27 1.27)) (justify left bottom))
   )
-  (label "IO0x*" (at 151.13 44.45 0)
-    (effects (font (size 1.27 1.27)) (justify left bottom))
-  )
