File: sch/Z80proto2/Z80proto2_IOblock.kicad_sch (KiCad schematic)
At the start: 31 parts, among them SW101 RESET, U101 LMC555, U11 V_TC6367, U14 AC541, U15 HC139, U17 TD62783, U18 TD62083, U21 23LC512, U4 HC138

Commit message: Add Async. FIFO support(EXPERIMENTAL)
Add FT245R Asynchronous FIFO support(EXPERIMENTAL)
change environment MiniLoader(zcc->sdcc)
Connections:
- net SPICS0*: now also U11.41 (PA6), U14.8 (A6); no longer U11.40 (PA5)
- net SPICS1*: now also U11.42 (PA7), U14.9 (A7); no longer U11.41 (PA6)
- net RXF*: now reaches U14.5 (A3)
- net TXE*: now reaches U14.7 (A5)
Changed lines of the file:
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@@
+    (stroke (width 0) (type default) (color 0 0 0 0))
+  )
+  (wire (pts (xy 52.07 328.93) (xy 39.37 328.93))
     (stroke (width 0) (type default) (color 0 0 0 0))
   )
@@
     (stroke (width 0) (type default) (color 0 0 0 0))
   )
+  (wire (pts (xy 39.37 323.85) (xy 52.07 323.85))
+    (stroke (width 0) (type default) (color 0 0 0 0))
+  )
   (polyline (pts (xy 113.03 78.74) (xy 113.03 162.56))
     (stroke (width 0) (type default) (color 0 0 0 0))
@@
     (stroke (width 0) (type default) (color 0 0 0 0))
   )
-  (wire (pts (xy 82.55 198.12) (xy 95.25 198.12))
+  (wire (pts (xy 82.55 200.66) (xy 95.25 200.66))
     (stroke (width 0) (type default) (color 0 0 0 0))
   )
@@
     (stroke (width 0) (type default) (color 0 0 0 0))
   )
+  (wire (pts (xy 52.07 326.39) (xy 39.37 326.39))
+    (stroke (width 0) (type default) (color 0 0 0 0))
+  )
   (wire (pts (xy 215.9 97.79) (xy 231.14 97.79))
     (stroke (width 0) (type default) (color 0 0 0 0))
@@
     (stroke (width 0) (type default) (color 0 0 0 0))
   )
+  (wire (pts (xy 39.37 318.77) (xy 52.07 318.77))
+    (stroke (width 0) (type default) (color 0 0 0 0))
+  )
   (wire (pts (xy 35.56 123.19) (xy 50.8 123.19))
     (stroke (width 0) (type default) (color 0 0 0 0))
@@
     (stroke (width 0) (type default) (color 0 0 0 0))
   )
-  (wire (pts (xy 82.55 200.66) (xy 95.25 200.66))
+  (wire (pts (xy 82.55 203.2) (xy 95.25 203.2))
     (stroke (width 0) (type default) (color 0 0 0 0))
   )
@@
     (effects (font (size 1.27 1.27)) (justify left bottom))
   )
-  (label "SPICS0*" (at 92.71 198.12 180)
+  (label "SPICS0*" (at 92.71 200.66 180)
     (effects (font (size 1.27 1.27)) (justify right bottom))
   )
@@
     (effects (font (size 1.27 1.27)) (justify left bottom))
   )
+  (label "SPICS0*" (at 41.91 326.39 0)
+    (effects (font (size 1.27 1.27)) (justify left bottom))
+  )
   (label "7seg_e" (at 81.28 275.59 0)
     (effects (font (size 1.27 1.27)) (justify left bottom))
@@
     (effects (font (size 1.27 1.27)) (justify left bottom))
   )
-  (label "SPICS1*" (at 92.71 200.66 180)
+  (label "SPICS1*" (at 92.71 203.2 180)
     (effects (font (size 1.27 1.27)) (justify right bottom))
   )
@@
     (effects (font (size 1.27 1.27)) (justify left bottom))
   )
+  (label "TXE*" (at 40.64 323.85 0)
+    (effects (font (size 1.27 1.27)) (justify left bottom))
+  )
   (label "D3" (at 38.1 134.62 0)
     (effects (font (size 1.27 1.27)) (justify left bottom))
@@
     (effects (font (size 1.27 1.27)) (justify left bottom))
   )
+  (label "RXF*" (at 40.64 318.77 0)
+    (effects (font (size 1.27 1.27)) (justify left bottom))
+  )
   (label "SPISI" (at 92.71 195.58 180)
     (effects (font (size 1.27 1.27)) (justify right bottom))
@@
     (effects (font (size 1.27 1.27)) (justify left bottom))
   )
+  (label "SPICS1*" (at 41.91 328.93 0)
+    (effects (font (size 1.27 1.27)) (justify left bottom))
+  )
